File: 27c322-adaptor/27c322.sch (KiCad schematic (older format))
At the start: 11 parts, among them P1 A19_SEL, P2 A18_SEL, P3 A20_SEL, Q1 MMBT3906, SW1 Switch_SPDT_x2, U1 27C4096, U2 27C322

Commit message: 27c322: Reduce R3 value to 1K in schematic
Parts:
- R3: value 10K -> 1K
Changed lines of the file:
@@
 P 3000 5350
 F 0 "R3" V 3080 5350 50  0000 C CNN
-F 1 "10K" V 3000 5350 50  0000 C CNN
+F 1 "1K" V 3000 5350 50  0000 C CNN
 F 2 "Resistors_SMD:R_0805_HandSoldering" V 2930 5350 50  0001 C CNN
 F 3 "" H 3000 5350 50  0000 C CNN
